Commit message: urdf: rename links, fix joint limits from MJCF with correct frame mapping
- Rename joints/links: yaw2roll→yaw2roll_left/right, hip_l→hip_left/right,
  leg→leg_left/right (and _2 variants)
- Fix all joint limits sourced from pollen-robotics/microduck robot_walk.xml
  with correct URDF-frame sign mapping (MJCF body quat vs URDF origin RPY)
- hip yaw: left -25°..+30°, right -25°..+30° (right axis is opposite → negated)
- ankles: ±90° (mapped from MJCF ±90°)
- head_yaw: ±170°, head_roll: ±25° (direct MJCF)
- knee/hip pitch/roll: ±90° / ±22° (symmetric, unchanged magnitude)
- Fix floating_base z offset so base_link sits on ground plane
- Replace package://microduck_description/meshes/ with ../meshes/ in .urdf only

File: urdf/microduck.common.xacro (robot description, xacro)
@@ -29,33 +29,33 @@
     <color rgba="0.039 0.047 0.055 1.0"/>
   </material>
-  <!-- Joint Limits (from MJCF) -->
-  <xacro:property name="left_hip_yaw_lower" value="-0.436"/>
-  <xacro:property name="left_hip_yaw_upper" value="0.524"/>
-  <xacro:property name="left_hip_roll_lower" value="-0.384"/>
-  <xacro:property name="left_hip_roll_upper" value="0.384"/>
-  <xacro:property name="left_hip_pitch_lower" value="-1.571"/>
-  <xacro:property name="left_hip_pitch_upper" value="1.571"/>
-  <xacro:property name="left_knee_lower" value="-2.094"/>
-  <xacro:property name="left_knee_upper" value="-0.035"/>
-  <xacro:property name="left_ankle_lower" value="-1.222"/>
-  <xacro:property name="left_ankle_upper" value="1.222"/>
-  <xacro:property name="right_hip_yaw_lower" value="-0.524"/>
-  <xacro:property name="right_hip_yaw_upper" value="0.436"/>
-  <xacro:property name="right_hip_roll_lower" value="-0.384"/>
-  <xacro:property name="right_hip_roll_upper" value="0.384"/>
-  <xacro:property name="right_hip_pitch_lower" value="-1.571"/>
-  <xacro:property name="right_hip_pitch_upper" value="1.571"/>
-  <xacro:property name="right_knee_lower" value="-2.094"/>
-  <xacro:property name="right_knee_upper" value="-0.035"/>
-  <xacro:property name="right_ankle_lower" value="-1.222"/>
-  <xacro:property name="right_ankle_upper" value="1.222"/>
-  <xacro:property name="neck_pitch_lower" value="-0.436"/>
-  <xacro:property name="neck_pitch_upper" value="0.873"/>
-  <xacro:property name="head_pitch_lower" value="-1.222"/>
-  <xacro:property name="head_pitch_upper" value="1.222"/>
-  <xacro:property name="head_yaw_lower" value="-1.222"/>
-  <xacro:property name="head_yaw_upper" value="1.222"/>
-  <xacro:property name="head_roll_lower" value="-0.611"/>
-  <xacro:property name="head_roll_upper" value="0.611"/>
+  <!-- Joint Limits from the upstream Microduck MJCF (source of truth) -->
+  <xacro:property name="left_hip_yaw_lower" value="-0.4363323129985824"/>
+  <xacro:property name="left_hip_yaw_upper" value="0.5235987755982988"/>
+  <xacro:property name="left_hip_roll_lower" value="-0.3839724354387525"/>
+  <xacro:property name="left_hip_roll_upper" value="0.3839724354387525"/>
+  <xacro:property name="left_hip_pitch_lower" value="-1.570796326795005"/>
+  <xacro:property name="left_hip_pitch_upper" value="1.5707963267947882"/>
+  <xacro:property name="left_knee_lower" value="-1.5707963267948966"/>
+  <xacro:property name="left_knee_upper" value="1.5707963267948966"/>
+  <xacro:property name="left_ankle_lower" value="-1.5707963267948912"/>
+  <xacro:property name="left_ankle_upper" value="1.5707963267949019"/>
+  <xacro:property name="right_hip_yaw_lower" value="-0.4363323129985824"/>
+  <xacro:property name="right_hip_yaw_upper" value="0.5235987755982988"/>
+  <xacro:property name="right_hip_roll_lower" value="-0.3839724354387525"/>
+  <xacro:property name="right_hip_roll_upper" value="0.3839724354387525"/>
+  <xacro:property name="right_hip_pitch_lower" value="-1.5707963267949268"/>
+  <xacro:property name="right_hip_pitch_upper" value="1.5707963267948664"/>
+  <xacro:property name="right_knee_lower" value="-1.5707963267948966"/>
+  <xacro:property name="right_knee_upper" value="1.5707963267948966"/>
+  <xacro:property name="right_ankle_lower" value="-1.5707963267948903"/>
+  <xacro:property name="right_ankle_upper" value="1.5707963267949028"/>
+  <xacro:property name="neck_pitch_lower" value="-1.5707963267948966"/>
+  <xacro:property name="neck_pitch_upper" value="1.0471975511965976"/>
+  <xacro:property name="head_pitch_lower" value="-1.5707963267948974"/>
+  <xacro:property name="head_pitch_upper" value="1.5707963267948957"/>
+  <xacro:property name="head_yaw_lower" value="-2.967059728390364"/>
+  <xacro:property name="head_yaw_upper" value="2.967059728390357"/>
+  <xacro:property name="head_roll_lower" value="-0.4363323129986037"/>
+  <xacro:property name="head_roll_upper" value="0.43633231299856107"/>
   <!-- Jaw joint limits (15th motor) -->
   <xacro:property name="jaw_lower" value="0.0"/>

File: urdf/microduck.joints.xacro (robot description, xacro)
@@ -5,8 +5,8 @@
       <parent link="base_link"/>
       <child link="trunk_base"/>
-      <origin xyz="0 0 0.12" rpy="0 0 0"/>
+      <origin xyz="0 0 0.105" rpy="0 0 0"/>
     </joint>
     <joint name="left_ankle" type="revolute">
-      <parent link="leg"/>
+      <parent link="leg_left"/>
       <child link="ankle_left"/>
       <origin xyz="0.0 0.042 -0.026" rpy="3.141593 -0.000000 0.000000"/>
@@ -17,5 +17,5 @@
     <joint name="left_knee" type="revolute">
       <parent link="upper_leg_left"/>
-      <child link="leg"/>
+      <child link="leg_left"/>
       <origin xyz="0.022 0.0357771 -0.004" rpy="3.141593 0.000000 1.570796"/>
       <axis xyz="0.0 0.0 1.0"/>
@@ -24,5 +24,5 @@
     </joint>
     <joint name="left_hip_pitch" type="revolute">
-      <parent link="hip_l"/>
+      <parent link="hip_left"/>
       <child link="upper_leg_left"/>
       <origin xyz="0.025 0.0 -0.0185" rpy="-1.570796 0.000000 -1.570796"/>
@@ -32,6 +32,6 @@
     </joint>
     <joint name="left_hip_roll" type="revolute">
-      <parent link="yaw2roll"/>
-      <child link="hip_l"/>
+      <parent link="yaw2roll_left"/>
+      <child link="hip_left"/>
       <origin xyz="0.0 0.0165 0.0125" rpy="-1.570796 0.000000 0.000000"/>
       <axis xyz="0.0 0.0 1.0"/>
@@ -64,5 +64,5 @@
     </joint>
     <joint name="right_ankle" type="revolute">
-      <parent link="leg_2"/>
+      <parent link="leg_right"/>
       <child link="ankle_right"/>
       <origin xyz="-0.042 0.0 -0.026" rpy="-3.141593 0.000000 1.570796"/>
@@ -73,5 +73,5 @@
     <joint name="right_knee" type="revolute">
       <parent link="upper_leg_right"/>
-      <child link="leg_2"/>
+      <child link="leg_right"/>
       <origin xyz="-0.022 0.0357771 -0.004" rpy="3.141593 0.000000 0.000000"/>
       <axis xyz="0.0 0.0 1.0"/>
@@ -80,5 +80,5 @@
     </joint>
     <joint name="right_hip_pitch" type="revolute">
-      <parent link="hip_l_2"/>
+      <parent link="hip_right"/>
       <child link="upper_leg_right"/>
       <origin xyz="0.025 0.0 -0.0185" rpy="-1.570796 0.000000 -1.570796"/>
@@ -88,6 +88,6 @@
     </joint>
     <joint name="right_hip_roll" type="revolute">
-      <parent link="yaw2roll_2"/>
-      <child link="hip_l_2"/>
+      <parent link="yaw2roll_right"/>
+      <child link="hip_right"/>
       <origin xyz="-0.0 0.0165 0.0125" rpy="1.570796 0.000000 3.141593"/>
       <axis xyz="0.0 0.0 1.0"/>
@@ -97,5 +97,5 @@
     <joint name="left_hip_yaw" type="revolute">
       <parent link="trunk_base"/>
-      <child link="yaw2roll"/>
+      <child link="yaw2roll_left"/>
       <origin xyz="0.006 0.0175 -0.005" rpy="-3.141593 0.000000 1.570796"/>
       <axis xyz="0.0 0.0 1.0"/>
@@ -113,5 +113,5 @@
     <joint name="right_hip_yaw" type="revolute">
       <parent link="trunk_base"/>
-      <child link="yaw2roll_2"/>
+      <child link="yaw2roll_right"/>
       <origin xyz="0.006 -0.0175 -0.005" rpy="3.141593 0.000000 1.570796"/>
       <axis xyz="0.0 0.0 1.0"/>

File: urdf/microduck.links.xacro (robot description, xacro)
@@ -38,6 +38,6 @@
       </inertial>
     </link>
-    <!-- leg -->
-    <link name="leg">
+    <!-- leg_left -->
+    <link name="leg_left">
       <visual>
         <origin xyz="-0.022 0.0357771 0.0385" rpy="1.570796 1.570796 0.000000"/>
@@ -103,6 +103,6 @@
       </inertial>
     </link>
-    <!-- hip_l -->
-    <link name="hip_l">
+    <!-- hip_left -->
+    <link name="hip_left">
       <visual>
         <origin xyz="0.021 0.0 -0.0185" rpy="1.570796 0.000000 1.570796"/>
@@ -125,6 +125,6 @@
       </inertial>
     </link>
-    <!-- yaw2roll -->
-    <link name="yaw2roll">
+    <!-- yaw2roll_left -->
+    <link name="yaw2roll_left">
       <visual>
         <origin xyz="-0.0175 -0.002 0.0125" rpy="3.141593 0.000000 0.000000"/>
@@ -419,6 +419,6 @@
       </inertial>
     </link>
-    <!-- leg_2 -->
-    <link name="leg_2">
+    <!-- leg_right -->
+    <link name="leg_right">
       <visual>
         <origin xyz="-0.042 0.0 -0.0115" rpy="-0.000000 -1.570796 0.000000"/>
@@ -484,6 +484,6 @@
       </inertial>
     </link>
-    <!-- hip_l_2 -->
-    <link name="hip_l_2">
+    <!-- hip_right -->
+    <link name="hip_right">
       <visual>
         <origin xyz="-0.0175 0.0 -0.0185" rpy="-1.570796 0.000000 0.000000"/>
@@ -506,6 +506,6 @@
       </inertial>
     </link>
-    <!-- yaw2roll_2 -->
-    <link name="yaw2roll_2">
+    <!-- yaw2roll_right -->
+    <link name="yaw2roll_right">
       <visual>
         <origin xyz="-0.0175 -0.002 0.0125" rpy="3.141593 0.000000 0.000000"/>

File: urdf/microduck.urdf (robot description, URDF)
Before this commit: robot microduck, 17 links, 16 joints
Links:
- removed link hip_l
- removed link hip_l_2
- removed link leg
- removed link leg_2
- removed link yaw2roll
- removed link yaw2roll_2
- added link hip_left, mass 0.01; visual mesh filename=../meshes/hip_l.stl scale=1.0 1.0 1.0; visual mesh filename=../meshes/seeed_bearing__configuration__22x16x4.stl scale=1.0 1.0 1.0
- added link hip_right, mass 0.01; visual mesh filename=../meshes/hip_l.stl scale=1.0 1.0 1.0; visual mesh filename=../meshes/seeed_bearing__configuration__22x16x4.stl scale=1.0 1.0 1.0
- added link leg_left, mass 0.01; visual mesh filename=../meshes/leg.stl scale=1.0 1.0 1.0; visual mesh filename=../meshes/xl330.stl scale=1.0 1.0 1.0
- added link leg_right, mass 0.01; visual mesh filename=../meshes/leg.stl scale=1.0 1.0 1.0; visual mesh filename=../meshes/xl330.stl scale=1.0 1.0 1.0
- added link yaw2roll_left, mass 0.01; visual mesh filename=../meshes/bearing_roll.stl scale=1.0 1.0 1.0; visual mesh filename=../meshes/seeed_bearing__configuration__22x16x4.stl scale=1.0 1.0 1.0
- added link yaw2roll_right, mass 0.01; visual mesh filename=../meshes/bearing_roll.stl scale=1.0 1.0 1.0; visual mesh filename=../meshes/seeed_bearing__configuration__22x16x4.stl scale=1.0 1.0 1.0
Joints:
- joint floating_base: origin xyz=0 0 0.12 rpy=0 0 0 -> xyz=0 0 0.105 rpy=0 0 0
- joint head_pitch: limit lower=-1.222 upper=1.222 effort=1.0 velocity=10.0 -> lower=-1.5707963267948974 upper=1.5707963267948957 effort=1.0 velocity=10.0
- joint head_roll: limit lower=-0.611 upper=0.611 effort=1.0 velocity=10.0 -> lower=-0.4363323129986037 upper=0.43633231299856107 effort=1.0 velocity=10.0
- joint head_yaw: limit lower=-1.222 upper=1.222 effort=1.0 velocity=10.0 -> lower=-2.967059728390364 upper=2.967059728390357 effort=1.0 velocity=10.0
- joint left_ankle: limit lower=-1.222 upper=1.222 effort=1.0 velocity=10.0 -> lower=-1.5707963267948912 upper=1.5707963267949019 effort=1.0 velocity=10.0; parent leg -> leg_left
- joint left_hip_pitch: limit lower=-1.571 upper=1.571 effort=1.0 velocity=10.0 -> lower=-1.570796326795005 upper=1.5707963267947882 effort=1.0 velocity=10.0; parent hip_l -> hip_left
- joint left_hip_roll: child hip_l -> hip_left; limit lower=-0.384 upper=0.384 effort=1.0 velocity=10.0 -> lower=-0.3839724354387525 upper=0.3839724354387525 effort=1.0 velocity=10.0; parent yaw2roll -> yaw2roll_left
- joint left_hip_yaw: child yaw2roll -> yaw2roll_left; limit lower=-0.436 upper=0.524 effort=1.0 velocity=10.0 -> lower=-0.4363323129985824 upper=0.5235987755982988 effort=1.0 velocity=10.0
- joint left_knee: child leg -> leg_left; limit lower=-2.094 upper=-0.035 effort=1.0 velocity=10.0 -> lower=-1.5707963267948966 upper=1.5707963267948966 effort=1.0 velocity=10.0
- joint neck_pitch: limit lower=-0.436 upper=0.873 effort=1.0 velocity=10.0 -> lower=-1.5707963267948966 upper=1.0471975511965976 effort=1.0 velocity=10.0
- joint right_ankle: limit lower=-1.222 upper=1.222 effort=1.0 velocity=10.0 -> lower=-1.5707963267948903 upper=1.5707963267949028 effort=1.0 velocity=10.0; parent leg_2 -> leg_right
- joint right_hip_pitch: limit lower=-1.571 upper=1.571 effort=1.0 velocity=10.0 -> lower=-1.5707963267949268 upper=1.5707963267948664 effort=1.0 velocity=10.0; parent hip_l_2 -> hip_right
- joint right_hip_roll: child hip_l_2 -> hip_right; limit lower=-0.384 upper=0.384 effort=1.0 velocity=10.0 -> lower=-0.3839724354387525 upper=0.3839724354387525 effort=1.0 velocity=10.0; parent yaw2roll_2 -> yaw2roll_right
- joint right_hip_yaw: child yaw2roll_2 -> yaw2roll_right; limit lower=-0.524 upper=0.436 effort=1.0 velocity=10.0 -> lower=-0.4363323129985824 upper=0.5235987755982988 effort=1.0 velocity=10.0
- joint right_knee: child leg_2 -> leg_right; limit lower=-2.094 upper=-0.035 effort=1.0 velocity=10.0 -> lower=-1.5707963267948966 upper=1.5707963267948966 effort=1.0 velocity=10.0
